Commit message: Add diff Gazebo controller plugin

File: urdf/car-robot-gazebo.xacro (robot description, xacro)
@@ -6,7 +6,28 @@
 	<xacro:macro name="color_wheel" params="x_position y_position">
 		<gazebo reference="${x_position}-${y_position}-wheel-link">
+		        <mu1>10000.0 </mu1>
+                        <mu2>10000.0 </mu2>
 			<material>Gazebo/Purple</material>
 		</gazebo>
 	</xacro:macro>
+	<gazebo>
+	<!-- differential drive control for Gazebo -->
+	<plugin name="differential_drive_controller" filename="libgazebo_ros_diff_drive.so">
+	<alwaysOn>true</alwaysOn>
+	<updateRate>100</updateRate>
+	<leftJoint>joint-chassis-rare-left-wheel</leftJoint>
+	<rightJoint>joint-chassis-rare-right-wheel</rightJoint>
+	<wheelSeparation>${chassis_width}</wheelSeparation>
+	<wheelDiameter>${2 * wheel_radius}</wheelDiameter>
+	<torque>0.1</torque>
+	<commandTopic>cmd_vel</commandTopic>
+	<odometryTopic>odom</odometryTopic>
+	<odometryFrame>odom</odometryFrame>
+	<robotBaseFrame>base_link</robotBaseFrame>
+	<publishWheelTF>true</publishWheelTF>
+	<publishOdom>true</publishOdom>
+	<publishWheelJointState>true</publishWheelJointState>
+	</plugin>
+	</gazebo>
 	<xacro:color_wheel x_position="front" y_position="right"/>
 	<xacro:color_wheel x_position="front" y_position="left" />

File: urdf/car-robot-params.xacro (robot description, xacro)
@@ -1,5 +1,5 @@
 <?xml version='1.0'?>
 <robot xmlns:xacro ="http://www.ros.org/wiki/xacro" >
-	<xacro:property name="chassis_length" value="0.2" />
+	<xacro:property name="chassis_length" value="0.14" />
 	<xacro:property name="chassis_width" value="0.12" />
 	<xacro:property name="chassis_height" value="0.01" />

File: urdf/car-robot-xacro.urdf (robot description, URDF)
Before this commit: robot car-robot, 6 links, 5 joints
Links:
- link chassis-link: geometry collision box size=0.14 0.12 0.01; visual box size=0.14 0.12 0.01
Joints:
- joint joint-chassis-front-left-wheel: origin xyz=0.06 -0.065 0 rpy=0 0 0 -> xyz=0.042 -0.065 0 rpy=0 0 0
- joint joint-chassis-front-right-wheel: origin xyz=0.06 0.065 0 rpy=0 0 0 -> xyz=0.042 0.065 0 rpy=0 0 0
- joint joint-chassis-rare-left-wheel: origin xyz=-0.06 -0.065 0 rpy=0 0 0 -> xyz=-0.042 -0.065 0 rpy=0 0 0
- joint joint-chassis-rare-right-wheel: origin xyz=-0.06 0.065 0 rpy=0 0 0 -> xyz=-0.042 0.065 0 rpy=0 0 0
